File: leakguard.kicad_pcb (KiCad board)
At the start: 4 copper layers, 99 x 90 mm, 123 parts, among them J101 Jack-DC, J102 Conn_01x05_Pin, J103 Conn_01x04_Pin, J104 Conn_01x02_Socket, J105 Conn_01x03_Socket, J201 Conn_01x05_Pin, J202 Conn_01x04_Pin, Q101 DMG1012UW, Q102 MMBT2222ALT1G, Q201 DMP2045U, SW101 RESET, SW102 IMPULSE, SW103 UNLOCK, SW201 RESET, SW202 PING, SW203 TEST, SW204 ADDRESS, U101 LMR50410, U102 AMS1117-3.3, U103 24LC512, U104 ESP32-C3_SUPERMINI_SMD, U105 STM32F746VETx, U106 W25Q32JVSS, U107 XL1278-SMT, U201 STM32L031K6Tx, U202 XL1278-SMT, Y101 16MHz, Y102 32768Hz, Y201 32.768kHz

Commit message: Final version sent to production
Parts:
- removed mouse-bite-2mm-slot (x2): VAL**, Panelization:mouse-bite-2mm-slot_1
- added D110: GREEN, LED_THT:LED_D3.0mm, F.Cu at (101.6, 66.5)
- added R119: 470, Resistor_SMD:R_0805_2012Metric_Pad1.20x1.40mm_HandSolder, B.Cu at (103.6, 65.8)
- C118, C119, C120, C121, C209, C210: value 10n -> 10p
- D109: footprint LED_THT:LED_D3.0mm -> LED_SMD:LED_0805_2012Metric_Pad1.15x1.40mm_HandSolder
- R118: value 470 -> 680; moved to F.Cu
- Y201: value 32.768kHz -> 32768Hz
- moved D109 23.1 mm to (116.1, 45.0), turned to 0 degrees
- moved R118 20.9 mm to (112.0, 45.0), turned to 180 degrees
- moved D108 6.35 mm to (108.0, 66.5)
- moved R117 6.35 mm to (110.0, 65.8)
- moved C201 0.78 mm to (82.8, 81.7)
Connections:
- U105 pad 32: unconnected-(U105-PC4-Pad32) -> /Main unit/LED_OK
Routing:
- net /Main unit/LED_OK: track 0.00 -> 43.2 mm, vias 0 -> 1
- net /Main unit/LED_IMP: track 62.0 -> 88.8 mm, vias 1 -> 2
- net GND: track 138.0 -> 113.0 mm, vias 46 -> 57
- net GNDBATT: track 78.1 -> 55.6 mm, vias 17 -> 19
- net /Main unit/QSPI_CLK: track 13.2 -> 29.8 mm, vias 2 -> 0
- net +12V: track 95.5 -> 103.8 mm, vias 3 -> 4
- net /Main unit/QSPI_IO0: track 24.5 -> 30.9 mm, vias 2 -> 0
- net /Main unit/LED_VALVE: track 51.9 -> 57.1 mm
- net /Main unit/QSPI_IO1: track 18.3 -> 23.3 mm, vias 2 -> 0
- net /Main unit/QSPI_IO2: track 25.6 -> 29.6 mm
- net /Main unit/LORA_DIO0: track 41.2 -> 38.0 mm
- net /Main unit/SWCLK: track 33.5 -> 36.5 mm
- net /Main unit/QSPI_NCS: track 28.3 -> 31.1 mm
- net /Main unit/RESET: track 81.4 -> 78.6 mm, vias 4 -> 3
- net /Main unit/QSPI_IO3: track 25.7 -> 28.2 mm, vias 2 -> 0
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Other:
- outline, holes or cut-outs redrawn
- board text added: "OK"
- board text added: "OLED"
- board text added: "SENSOR"
- board text added: "VALVE"
- board text removed: "JLCJLCJLCJLC"
- board text removed: "VALVE CLS"
