File: main.kicad_sch (KiCad schematic)
At the start: 79 parts, among them J101 Jack-DC, J102 Conn_01x05_Pin, J103 Conn_01x04_Pin, J104 Conn_01x02_Socket, J105 Conn_01x03_Socket, Q101 DMG1012UW, Q102 MMBT2222ALT1G, SW101 RESET, SW102 IMPULSE, SW103 UNLOCK, U101 LMR50410, U102 AMS1117-3.3, U103 24LC512, U104 ESP32-C3_SUPERMINI_SMD, U105 STM32F746VETx, U106 W25Q32JVSS, U107 XL1278-SMT, Y101 16MHz, Y102 32768Hz

Commit message: Final version sent to production
Parts:
- added D110: GREEN, LED_THT:LED_D3.0mm, symbol Device:LED
- added R119: 470, Resistor_SMD:R_0805_2012Metric_Pad1.20x1.40mm_HandSolder, symbol Device:R
- C118, C119, C120, C121: value 10n -> 10p
- D109: footprint LED_THT:LED_D3.0mm -> LED_SMD:LED_0805_2012Metric_Pad1.15x1.40mm_HandSolder
- R118: value 470 -> 680
Connections:
- net GND: now also R119.2
- net LED_OK: now reaches U105.32 (PC4)
- net LED_OK: now also D110.2 (A)
- new net: D110.1 (K), R119.1
Other:
- moved on the sheet: TP102
