File: sensor.kicad_sch (KiCad schematic)
At the start: 33 parts, among them J201 Conn_01x05_Pin, J202 Conn_01x04_Pin, Q201 DMP2045U, SW201 RESET, SW202 PING, SW203 TEST, SW204 ADDRESS, U201 STM32L031K6Tx, U202 XL1278-SMT, Y201 32.768kHz

Commit message: Final version sent to production
Parts:
- C209, C210: value 10n -> 10p
- Y201: value 32.768kHz -> 32768Hz
Changed lines of the file:
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@@
 			)
 		)
-		(property "Value" "32.768kHz"
+		(property "Value" "32768Hz"
 			(at 43.18 87.884 0)
 			(effects
@@
 			)
 		)
-		(property "Value" "10n"
+		(property "Value" "10p"
 			(at 29.972 102.87 0)
 			(effects
@@
 			)
 		)
-		(property "Value" "10n"
+		(property "Value" "10p"
 			(at 53.848 100.33 0)
 			(effects
